File: Adafruit TFP401 to 40pin TFT.sch (EAGLE design)
At the start: 90 parts, among them IC1 AR1100_SSOP, Q1 BSS138, U1 TFP401, U2 24LC02BT-I/OT, U3 LT1117(3V3), U4 FAN5333BSX, X1 47151-0001, X2 microUSB, X3 XF2-40-RARBT, Y1 12MHz

Commit message: Модификация платы
Parts:
- removed FID2: FIDUCIAL"", microbuilder:FIDUCIAL""
- removed U$31, U$32, U$33, U$34: MOUNTINGHOLE3.0, microbuilder:MOUNTINGHOLE3.0
- removed X2: microUSB, microbuilder:USBMICRO_20329
- added X4: MINI-USB-32005-201, con-cypressindustries:MINI-USB-32005-201
- U2: device microbuilder:EEPROM_I2C_MCP24AA32 -> microchip:24C02ASM
Connections:
- net D+: now also X4.3; no longer X2.D+
- net D-: now also X4.2; no longer X2.D-
- net GND: now also X4.5; no longer X2.GND
- net VIN: now also X4.1; no longer X2.VBUS
Other:
- moved on the sheet: C20, R3, R4
